File: hardware/hub-carrier-p4.sch (EAGLE design)
At the start: 66 parts, among them J10 43045-0412 ECU, J11 43045-0412 CHAIN, J12 GPS 1x5 2.54, J13 TO DEVKIT POE_PWR1, U1 D36V28F5, U2 TJA1051T/3, U3 SN65HVD230DR, U4 ESP32-P4-DevKit, U5 DS3231SN#, U6 ESP32-C6-MINI-1-N4

Commit message: P4 hub carrier on the Waveshare ESP32-P4-WIFI6, with an Adafruit GPS and external antenna
The second hub schematic moves from the Olimex ESP32-P4-DevKit to the
Waveshare ESP32-P4-WIFI6 (SKU 32020), which carries its own ESP32-C6
Wi-Fi. The carrier loses its Wi-Fi module, the SDIO pull-ups, the C6
programming lines and the POE_PWR1 lead:

- the board's 5 V goes into VSYS through D3, as on the C6 carrier;
  VBUS (its USB 5 V) is left unconnected
- CAN, 12 V sense and the clock's I2C stay on the same GPIOs; the
  clock's 1 Hz line moves to GPIO31
- J12 is now a 9-way socket for the Adafruit Ultimate GPS (product
  746), with standoff holes from Adafruit's board file and an external
  active antenna through a u.FL-to-SMA lead in the case wall
- Q1 lets GPIO50 switch the GPS off, since its enable pin sits at 5 V

The Waveshare footprint is the Raspberry Pi Pico pin pattern with the
board's outline and antenna notch from Waveshare's drawings. Electrical
spec section 5, the PCBWay list and the drawing are updated. The Olimex
version stays in the history (4ca940c).

Co-Authored-By: Claude Opus 5.5 <noreply@anthropic.com>
Parts:
- removed C11: 10u 25V, haltech-gauges:C0805
- removed C12, C13: 100n, haltech-gauges:C0805
- removed J13: TO DEVKIT POE_PWR1, haltech-gauges:POWER-2
- removed JP3: GPS 3V3/5V, haltech-gauges:JUMPER-3
- removed R10, R11, R12, R13, R14, R15, R16, R17: 10k, haltech-gauges:R0805
- removed TP6: C6 EN, haltech-gauges:TESTPOINT
- removed TP7: C6 TXD, haltech-gauges:TESTPOINT
- removed TP8: C6 RXD, haltech-gauges:TESTPOINT
- removed TP9: C6 BOOT, haltech-gauges:TESTPOINT
- removed U6: ESP32-C6-MINI-1-N4, haltech-gauges:ESP32-C6-MINI-1
- added D3: SS14, haltech-gauges:SCHOTTKY-SMA
- added Q1: 2N7002, haltech-gauges:2N7002
- added R24: 100k, haltech-gauges:R0805
- J12: value GPS 1x5 2.54 -> ADAFRUIT 746 SOCKET; device haltech-gauges:GPS-HEADER -> haltech-gauges:ADAFRUIT-ULTIMATE-GPS
- U4: value ESP32-P4-DevKit -> ESP32-P4-WIFI6; device haltech-gauges:OLIMEX-ESP32-P4-DEVKIT -> haltech-gauges:WAVESHARE-ESP32-P4-WIFI6
Connections:
- removed net C6_BOOT: R16.2, TP9.TP, U4.IO53, U6.IO9
- removed net C6_EN: C13.1, R10.2, TP6.TP, U4.IO54, U6.EN
- removed net C6_IO8: R17.2, U6.IO8
- removed net C6_RXD: TP8.TP, U4.IO4, U6.RXD0
- removed net C6_TXD: TP7.TP, U4.IO5, U6.TXD0
- removed net C6_WAKE: U4.IO6, U6.IO2
- removed net GPS_RXD: J12.RXD, U4.IO11
- removed net GPS_TXD: J12.TXD, R22.1
- removed net GPS_VCC: C16.1, J12.VCC, JP3.2
- removed net SDIO_CLK: U4.IO18, U6.IO19
- removed net SDIO_CMD: R11.2, U4.IO19, U6.IO18
- removed net SDIO_D0: R12.2, U4.IO14, U6.IO20
- removed net SDIO_D1: R13.2, U4.IO15, U6.IO21
- removed net SDIO_D2: R14.2, U4.IO16, U6.IO22
- removed net SDIO_D3: R15.2, U4.IO17, U6.IO23
- new net +5V_MCU: D3.K, U4.VSYS
- new net GPS_EN: J12.EN, Q1.D
- new net GPS_OFF: Q1.G, R24.1, U4.IO50
- new net GPS_TX: J12.TX, R22.1
- new net GPS_TX_IN: R22.2, U4.IO28
- net +3V3: no longer C11.1, C12.1, JP3.1, R10.1, R11.1, R12.1, R13.1, R14.1, R15.1, R16.1, R17.1, U6.3V3
- net +5V: now also C16.1, D3.A, J12.VIN; no longer J13.+5V, JP3.3
- net GND: now also Q1.S, R24.2, U4.GND@5, U4.GND@6, U4.GND@7, U4.GND@8; no longer C11.2, C12.2, C13.2, J13.GND, U6.GND@1, U6.GND@11, U6.GND@14, U6.GND@2, U6.GND@36, U6.GND@37, U6.GND@38, U6.GND@39, U6.GND@40, U6.GND@41, U6.GND@42, U6.GND@43, U6.GND@44, U6.GND@45, U6.GND@46, U6.GND@47, U6.GND@48, U6.GND@49, U6.GND@50, U6.GND@51, U6.GND@52, U6.GND@53
- net GPS_PPS_IN: now also U4.IO30; no longer U4.IO12
- net GPS_RX: now also J12.RX, U4.IO29; no longer R22.2, U4.IO10
- net RST: now also U4.RUN; no longer U4.EN
- net RTC_INT: now also U4.IO31; no longer U4.IO9
Other:
- note added: "Footprints are generic or placeholders, except U4's pins and outline and J12's pins and holes, which come from the makers' files."
- note added: "Haltech gauges: hub carrier, ESP32-P4 variant (Waveshare ESP32-P4-WIFI6)"
- note added: "Its Wi-Fi (an ESP32-C6) is on the board, with the antenna at the far end: keep the carrier's copper away from that end."
- note added: "J12 takes an Adafruit Ultimate GPS (product 746) by its 9-pin header. It uses an external active antenna, through a u.FL-to-SMA lead to a socket in the case."
- note added: "Q1 turns the GPS off while GPIO50 is high (it pulls the GPS board's EN low); R24 keeps the GPS on while the P4 is in reset."
- note added: "The carrier's 5 V reaches the board's VSYS pin through D3. Never connect VBUS (pin 40): it is the board's USB 5 V."
- note added: "U4 is the Waveshare ESP32-P4-WIFI6 (SKU 32020) on two 1x20 sockets: Raspberry Pi Pico pin pattern, USB-C end at pins 1 and 40."
- note added: "U5 is the clock, on the board's own I2C bus (GPIO7, GPIO8; 2.2 k pull-ups on the board). BT1 is a CR2032; fit JP2 only with a rechargeable ML2032."
- note removed: "Do not feed the DevKit through EXT2-1 (+5V): with USB plugged in, that pin back-feeds the PC."
- note removed: "Haltech gauges: hub carrier, ESP32-P4 variant (Olimex ESP32-P4-DevKit)"
- note removed: "J12 is the optional GPS header: 1 VCC (JP3 picks 3.3 V or 5 V), 2 GND, 3 TXD from the module, 4 RXD to it, 5 PPS."
- note removed: "J13 feeds the DevKit: wire J13-1 to POE_PWR1 pin 4 (+5VP) and J13-2 to pin 3 (GND). Leave POE_PWR1 pins 1 and 2 open."
- note removed: "The DevKit already has 2.2 k pull-ups on SDA and SCL (GPIO7, GPIO8). Footprints are generic or placeholders."
- note removed: "U4 is the Olimex ESP32-P4-DevKit (rev C), pins down, USB-C end at EXT pin 1. It takes its 3.3 V rail to the carrier on EXT1-1."
- note removed: "U5 is the clock. BT1 is a CR2032; fit JP2 only with a rechargeable ML2032, never with a CR2032."
- note removed: "U6 is the Wi-Fi radio (ESP-Hosted over SDIO, the pins Espressif's own P4 board uses). Antenna at a board edge, no copper under it."
- moved on the sheet: BT1, C10, C14, C15, C16, C6, C7, C8, D6, JP2, R1, R2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
